Commit message: fix: disabled heatcam and fixed sock physics

File: description/urdf/sock.urdf.xacro (robot description, xacro)
@@ -1,13 +1,41 @@
 <?xml version="1.0"?>
-<robot name="socks" xmlns:xacro="http://www.ros.org/wiki/xacro">
+<robot name="sock" xmlns:xacro="http://www.ros.org/wiki/xacro">
   <link name="sock">
-<!--     <collision>
-      <origin xyz="0 0 0" rpy="0 0 0" />
+    <collision>
+      <!-- POSE 1 -->
+      <origin xyz="11.0358938 -8.6 5.1" rpy="1.57 0 -1.57" />
+      <!-- POSE 2 -->
+      <!-- <origin xyz="11.0358938 -8.6 5.1" rpy="0 0 1.57" /> -->
+      <!-- POSE 3 -->
+      <!-- <origin xyz="11.0358938 -8.6 5.1" rpy="-1.57 0 0" /> -->
+      <!-- POSE 4 -->
+      <!-- <origin xyz="11.0358938 -8.6 5.1" rpy="0.2 0.2 1.57" /> -->
       <geometry>
         <mesh filename="package://isaac_description/meshes/sock.dae"/>
       </geometry>
-    </collision> -->
+      <surface>
+        <friction>
+          <ode>
+           <mu>0.8</mu>
+           <mu2>0.8</mu2>
+          </ode>
+        </friction>
+        <contact>
+          <ode>
+            <soft_cfm>0.01</soft_cfm>
+            <soft_erp>0.2</soft_erp>
+          </ode>
+        </contact>
+      </surface>
+    </collision>
     <visual>
-      <origin xyz="0 0 0" rpy="0 0 0" />
+      <!-- POSE 1 -->
+      <origin xyz="11.0358938 -8.6 5.1" rpy="1.57 0 -1.57" />
+      <!-- POSE 2 -->
+      <!-- <origin xyz="11.0358938 -8.6 5.1" rpy="0 0 1.57" /> -->
+      <!-- POSE 3 -->
+      <!-- <origin xyz="11.0358938 -8.6 5.1" rpy="-1.57 0 0" /> -->
+      <!-- POSE 4 -->
+      <!-- <origin xyz="11.0358938 -8.6 5.1" rpy="0.2 0.2 1.57" /> -->
       <geometry>
         <mesh filename="package://isaac_description/meshes/sock.dae"/>
@@ -15,10 +43,16 @@
     </visual>
     <inertial>
-      <mass value="100" />
-      <origin xyz="0 0 0" rpy="0 0 0" />
-      <inertia ixx="1" ixy="0" ixz="0" iyy="1" iyz="0" izz="1" />
+      <mass value="0.05" />
+      <!-- POSE 1 -->
+      <origin xyz="11.0358938 -8.6 5.1" rpy="1.57 0 -1.57" />
+      <!-- POSE 2 -->
+      <!-- <origin xyz="11.0358938 -8.6 5.1" rpy="0 0 1.57" /> -->
+      <!-- POSE 3 -->
+      <!-- <origin xyz="11.0358938 -8.6 5.1" rpy="-1.57 0 0" /> -->
+      <!-- POSE 4 -->
+      <!-- <origin xyz="11.0358938 -8.6 5.1" rpy="0.2 0.2 1.57" /> -->
+      <inertia ixx="0.00004" ixy="0" ixz="0" iyy="0.0004" iyz="0" izz="0.0004" />
     </inertial>
   </link>
-  <!-- tf publisher -->
   <gazebo>
     <plugin name="truth_ros" filename="libgazebo_model_plugin_truth.so">
@@ -31,4 +65,10 @@
       <static>false</static>
     </plugin>
+    <material>Gazebo/Blue</material>
+    <mu>0.8</mu>
+    <mu2>0.8</mu2>
+    <minDepth>0.001</minDepth>
+    <kp>1000.0</kp>
+    <kd>100.0</kd>
   </gazebo>
 </robot>
